Commit message: Added jammer links

File: vega4_description/urdf/vega4.urdf.xacro (robot description, xacro)
@@ -33,4 +33,48 @@
     </visual>
     </link>
+    <joint name="jammer_gantry_joint" type="fixed">
+      <parent link="gantry_upper_link"/>
+      <child link="jammer_link"/>
+      <origin xyz="0.05 0 0" rpy="0 0 0"/>
+      <axis xyz="0 0 1"/>
+    </joint>
+    <link name="jammer_link">
+      <visual>
+        <geometry>
+          <box size="0.03 0.01 0.01"/>
+        </geometry>
+        <origin xyz="0.015 0 0" rpy="0 0 0"/>
+      </visual>
+    </link>
+    <joint name="jammer_shoulder_joint" type="revolute">
+      <parent link="jammer_link"/>
+      <child link="jammer_shoulder_link"/>
+      <origin xyz="0.05 0 0" rpy="0 0 0"/>
+      <axis xyz="0 0 1"/>
+      <limit lower="${-((M_PI/2)+M_PI/6)}" upper="${(M_PI/2)+M_PI/6}" effort="2" velocity="0.3"/>
+    </joint>
+    <link name="jammer_shoulder_link">
+      <visual>
+        <geometry>
+          <box size="0.03 0.01 0.01"/>
+        </geometry>
+        <origin xyz="0.015 0 0" rpy="0 0 0"/>
+      </visual>
+    </link>
+    <joint name="jammer_elbow_joint" type="revolute">
+      <parent link="jammer_shoulder_link"/>
+      <child link="jammer_elbow_link"/>
+      <origin xyz="0.05 0 0" rpy="0 0 0"/>
+      <axis xyz="0 0 1"/>
+      <limit lower="${-((M_PI/2)+M_PI/6)}" upper="${(M_PI/2)+M_PI/6}" effort="2" velocity="0.3"/>
+    </joint>
+    <link name="jammer_elbow_link">
+      <visual>
+        <geometry>
+          <box size="0.03 0.01 0.01"/>
+        </geometry>
+        <origin xyz="0.015 0 0" rpy="0 0 0"/>
+      </visual>
+    </link>
     <joint name="head_joint" type="revolute">
       <parent link="gantry_upper_link"/>

Commit message: Add urdf to standard vega launch and connect camera_link to head

File: vega4_description/urdf/vega4.urdf.xacro (robot description, xacro)
@@ -94,9 +94,9 @@
     <joint name="head_camera_joint" type="fixed">
       <parent link="head_link"/>
-      <child link="head_camera_link"/>
+      <child link="camera_link"/>
       <origin xyz="0 0 0" rpy="0 0 0"/>
       <axis xyz="0 0 1"/>
     </joint>
-    <link name="head_camera_link">
+    <link name="camera_link">
       <visual>
         <geometry>

Commit message: Launch files and meshes

File: vega4_description/urdf/vega4.urdf.xacro (robot description, xacro)
@@ -7,5 +7,5 @@
       <parent link="base_link"/>
       <child link="gantry_lower_link"/>
-      <origin xyz="0 0 0" rpy="0 0 0"/>
+      <origin xyz="-0.05 0 0.13" rpy="0 0 0"/>
       <axis xyz="0 0 1"/>
     </joint>
@@ -13,7 +13,7 @@
       <visual>
         <geometry>
-          <box size="0.1 0.1 0.6"/>
+          <mesh scale="0.001 0.001 0.001" filename="package://vega4_description/meshes/gantry_lower_link.stl" />
         </geometry>
-        <origin xyz="0 0 0.3" rpy="0 0 0"/>
+        <origin xyz="0 0 0" rpy="${M_PI/2} 0 ${M_PI/2}"/>
       </visual>
     </link>
@@ -21,5 +21,5 @@
       <parent link="gantry_lower_link"/>
       <child link="gantry_upper_link"/>
-      <origin xyz="0 0 0.25" rpy="0 0 0"/>
+      <origin xyz="0 0 0.01" rpy="0 0 0"/>
       <axis xyz="0 0 1"/>
       <limit lower="0.0" upper="0.5" effort="2" velocity="0.3"/>
@@ -28,7 +28,7 @@
     <visual>
       <geometry>
-        <cylinder radius="0.05" length="0.5"/>
+        <mesh scale="0.001 0.001 0.001" filename="package://vega4_description/meshes/gantry_upper_link.stl" />
       </geometry>
-      <origin xyz="0 0 0.1" rpy="0 0 0"/>
+      <origin xyz="0 0 -0.26" rpy="${M_PI/2} 0 ${M_PI/2}"/>
     </visual>
     </link>
@@ -42,7 +42,7 @@
       <visual>
         <geometry>
-          <box size="0.03 0.01 0.01"/>
+          <mesh scale="0.001 0.001 0.001" filename="package://vega4_description/meshes/jammer_link.stl" />
         </geometry>
-        <origin xyz="0.015 0 0" rpy="0 0 0"/>
+        <origin xyz="0 0 0" rpy="${M_PI/2} 0 ${M_PI/2}"/>
       </visual>
     </link>
@@ -57,7 +57,7 @@
       <visual>
         <geometry>
-          <box size="0.03 0.01 0.01"/>
+          <mesh scale="0.001 0.001 0.001" filename="package://vega4_description/meshes/jammer_shoulder_link.stl" />
         </geometry>
-        <origin xyz="0.015 0 0" rpy="0 0 0"/>
+        <origin xyz="0 0 0" rpy="${M_PI/2} 0 ${M_PI/2}"/>
       </visual>
     </link>
@@ -72,7 +72,7 @@
       <visual>
         <geometry>
-          <box size="0.03 0.01 0.01"/>
+          <mesh scale="0.001 0.001 0.001" filename="package://vega4_description/meshes/jammer_elbow_link.stl" />
         </geometry>
-        <origin xyz="0.015 0 0" rpy="0 0 0"/>
+        <origin xyz="0 0 0" rpy="${M_PI/2} 0 ${M_PI/2}"/>
       </visual>
     </link>
@@ -87,7 +87,7 @@
       <visual>
         <geometry>
-          <box size="0.05 0.3 0.1"/>
+          <mesh scale="0.001 0.001 0.001" filename="package://vega4_description/meshes/head_link.stl" />
         </geometry>
-        <origin xyz="0 0 0" rpy="0 0 0"/>
+        <origin xyz="0 0 0" rpy="${M_PI/2} 0 ${M_PI/2}"/>
       </visual>
     </link>
@@ -103,5 +103,5 @@
           <box size="0.1 0.05 0.05"/>
         </geometry>
-        <origin xyz="0 0 0" rpy="0 0 0"/>
+        <origin xyz="0 0 0" rpy="${M_PI/2} 0 ${M_PI/2}"/>
       </visual>
     </link>

Commit message: URDF mostly complete

File: vega4_description/urdf/vega4.urdf.xacro (robot description, xacro)
@@ -16,4 +16,8 @@
         </geometry>
         <origin xyz="0 0 0" rpy="${M_PI/2} 0 ${M_PI/2}"/>
+      <material name="Metal">
+        <!--<color rgba="0 1.0 0 1"/>-->
+        <texture filename="package://vega4_description/material/metal.jpg"/>
+      </material>
       </visual>
     </link>
@@ -21,5 +25,5 @@
       <parent link="gantry_lower_link"/>
       <child link="gantry_upper_link"/>
-      <origin xyz="0 0 0.01" rpy="0 0 0"/>
+      <origin xyz="0.03 0 0.01" rpy="0 0 0"/>
       <axis xyz="0 0 1"/>
       <limit lower="0.0" upper="0.5" effort="2" velocity="0.3"/>
@@ -30,5 +34,9 @@
         <mesh scale="0.001 0.001 0.001" filename="package://vega4_description/meshes/gantry_upper_link.stl" />
       </geometry>
-      <origin xyz="0 0 -0.26" rpy="${M_PI/2} 0 ${M_PI/2}"/>
+      <origin xyz="0 0 0" rpy="${M_PI/2} 0 ${M_PI/2}"/>
+      <material name="Wood">
+        <!--<color rgba="0 1.0 0 1"/>-->
+        <texture filename="package://vega4_description/material/wood.jpg"/>
+      </material>
     </visual>
     </link>
@@ -36,5 +44,5 @@
       <parent link="gantry_upper_link"/>
       <child link="jammer_link"/>
-      <origin xyz="0.05 0 0" rpy="0 0 0"/>
+      <origin xyz="0.0075 0 0.1" rpy="0 0 0"/>
       <axis xyz="0 0 1"/>
     </joint>
@@ -45,4 +53,5 @@
         </geometry>
         <origin xyz="0 0 0" rpy="${M_PI/2} 0 ${M_PI/2}"/>
+      <material name="Black"/>
       </visual>
     </link>
@@ -50,5 +59,5 @@
       <parent link="jammer_link"/>
       <child link="jammer_shoulder_link"/>
-      <origin xyz="0.05 0 0" rpy="0 0 0"/>
+      <origin xyz="0.044 0 0" rpy="0 0 0"/>
       <axis xyz="0 0 1"/>
       <limit lower="${-((M_PI/2)+M_PI/6)}" upper="${(M_PI/2)+M_PI/6}" effort="2" velocity="0.3"/>
@@ -60,4 +69,7 @@
         </geometry>
         <origin xyz="0 0 0" rpy="${M_PI/2} 0 ${M_PI/2}"/>
+      <material name="Grey">
+        <color rgba="0.3 0.3 0.3 1"/>
+      </material>
       </visual>
     </link>
@@ -65,5 +77,5 @@
       <parent link="jammer_shoulder_link"/>
       <child link="jammer_elbow_link"/>
-      <origin xyz="0.05 0 0" rpy="0 0 0"/>
+      <origin xyz="0.1075 0 0" rpy="0 0 0"/>
       <axis xyz="0 0 1"/>
       <limit lower="${-((M_PI/2)+M_PI/6)}" upper="${(M_PI/2)+M_PI/6}" effort="2" velocity="0.3"/>
@@ -75,4 +87,5 @@
         </geometry>
         <origin xyz="0 0 0" rpy="${M_PI/2} 0 ${M_PI/2}"/>
+        <material name="Metal"/>
       </visual>
     </link>
@@ -80,7 +93,7 @@
       <parent link="gantry_upper_link"/>
       <child link="head_link"/>
-      <origin xyz="0 0 0.5" rpy="0 0 0"/>
-      <axis xyz="0 -1 0"/>
-      <limit lower="${-M_PI/6}" upper="${M_PI}" effort="2" velocity="0.3"/>
+      <origin xyz="-0.025 0 0.578" rpy="0 0 0"/>
+      <axis xyz="0 1 0"/>
+      <limit lower="${M_PI/6}" upper="${-M_PI}" effort="2" velocity="0.3"/>
     </joint>
     <link name="head_link">
@@ -89,5 +102,8 @@
           <mesh scale="0.001 0.001 0.001" filename="package://vega4_description/meshes/head_link.stl" />
         </geometry>
-        <origin xyz="0 0 0" rpy="${M_PI/2} 0 ${M_PI/2}"/>
+        <origin xyz="0 0 0" rpy="${M_PI/2} ${-M_PI/2} ${M_PI}"/>
+        <material name="Black">
+          <color rgba="0 0 0 0.9"/>
+        </material>
       </visual>
     </link>
@@ -95,14 +111,8 @@
       <parent link="head_link"/>
       <child link="camera_link"/>
-      <origin xyz="0 0 0" rpy="0 0 0"/>
+      <origin xyz="0.08 0 -0.015" rpy="0 0 0"/>
       <axis xyz="0 0 1"/>
     </joint>
     <link name="camera_link">
-      <visual>
-        <geometry>
-          <box size="0.1 0.05 0.05"/>
-        </geometry>
-        <origin xyz="0 0 0" rpy="${M_PI/2} 0 ${M_PI/2}"/>
-      </visual>
     </link>
   </xacro:macro>
